File: MuReSC_GaN_v1/Project.kicad_pcb (KiCad board)
At the start: 4 copper layers, 69.3 x 40 mm, 115 parts, among them IC1 STM32G474RET6, IC10 UCC12040DVE, IC11 LMG1020YFFR, IC12 LMG1020YFFR, IC13 LMG1020YFFR, IC14 LMG1020YFFR, IC2 TPSM5601R5HRDAR, IC3 ISO7720FQDQ1, IC4 ISO7720FQDQ1, IC5 ISO7720FQDQ1, IC6 ISO7720FQDQ1, IC7 UCC12040DVE, IC8 UCC12040DVE, IC9 UCC12040DVE, J1 62000211121_x6, J2 62000211121, J3 62000211121_x1, J4 62000211121_x1, P1 691214110002, P2 691214110002, Q1 GS61004B-TR, Q2 GS61004B-TR, Q3 GS61004B-TR, Q4 GS61004B-TR, Y1 NX3215SA-32.768K-STD-MUS-2, Y2 NX3225SA-24.000MHZ-STD-CSR-1

Commit message: quasi finito
Parts:
- removed RS5, RS6: R, Resistor_SMD:R_0603_1608Metric_Pad0.98x0.95mm_HandSolder
- removed Z4: TSZU52C3V3_RGG, SamacSys_Parts:TSZU52C3V3RGG
- C3, RS7, RS8, Z3: moved to B.Cu
- moved P2 131.7 mm to (81.8, 88.4), turned to 90 degrees
- moved C3 126.0 mm to (77.2, 86.9), turned to 90 degrees
- moved C1 106.3 mm to (83.1, 98.3)
- moved L1 105.7 mm to (83.3, 108.7), turned to -90 degrees
- moved C2 99.6 mm to (77.0, 105.1)
- moved RS8 90.9 mm to (68.5, 81.0), turned to 0 degrees
- moved RS7 86.2 mm to (71.8, 81.2), turned to 0 degrees
- moved Z3 86.1 mm to (72.0, 83.6), turned to 0 degrees
- moved Z2 71.0 mm to (35.9, 116.1), turned to 180 degrees
- moved RS4 67.3 mm to (33.0, 116.6)
- moved RS3 66.4 mm to (35.8, 118.4), turned to 180 degrees
- moved RS2 66.0 mm to (28.6, 117.3), turned to 180 degrees
- moved Z1 64.6 mm to (28.3, 115.1), turned to 180 degrees
- moved RS1 61.8 mm to (31.2, 116.7), turned to -90 degrees
- moved J4 6.39 mm to (23.1, 117.9)
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Connections:
- net Net-(C1-Pad2) renamed /CENTER
- IC1 pad 21: /COMP2_INP -> /ADC2_IN2
Routing:
- net /S2: track 64.9 -> 150.9 mm, vias 4 -> 35
- net /ADC2_IN2: track 0.00 -> 67.4 mm, vias 0 -> 3
- net GND: track 300.1 -> 337.8 mm, vias 216 -> 256
- net /COMP1_INP: track 0.00 -> 25.6 mm, vias 0 -> 3
- net /ADC1_IN1: track 0.00 -> 18.9 mm, vias 0 -> 2
- net /S1: track 58.3 -> 75.4 mm, vias 4 -> 35
- net /VDDI2: track 16.0 -> 25.1 mm, vias 4 -> 8
- net /VDDI1: track 19.5 -> 25.9 mm, vias 4 -> 8
- net /COMP2_INM: track 9.31 -> 15.5 mm
- net /COMP1_INM: track 12.4 -> 18.5 mm
- net /VDD48V: track 1.34 -> 5.00 mm
- net Net-(CFT2-OUT): track 0.00 -> 2.24 mm
- net Net-(CFT1-OUT): track 0.00 -> 2.10 mm
- net /VDDI4: track 24.5 -> 25.1 mm
- net /S3: vias 6 -> 36
- added copper zone on F.Cu, net /CENTER
- added copper zone on F.Cu, net /S1
- added copper zone on F.Cu, net /S2
- added copper zone on In2.Cu, net /S2
- added copper zone on F.Cu, net /VDDI1
- added copper zone on In2.Cu, net /VDDI1
- added copper zone on F.Cu, net /VDDI2
- added copper zone on In2.Cu, net /VDDI2
Other:
- board size 69.3 x 40 mm -> 71.1 x 40 mm

Commit message: LAYOUT DRC
Parts:
- COL1, COL2: footprint Capacitor_SMD:C_0201_0603Metric_Pad0.64x0.40mm_HandSolder -> SamacSys_Parts:CAPC0603X33N
- moved J4 0.25 mm to (23.1, 117.6)
Routing:
- net /T_SWCLK: track 29.9 -> 22.7 mm
- net /T_SWDIO: track 30.1 -> 24.8 mm
- net /VDD5V: track 30.9 -> 36.1 mm, vias 45 -> 37
- net GND: track 337.8 -> 333.4 mm, vias 256 -> 232
- net /UBUTT: track 30.5 -> 29.9 mm
- net /S3: track 68.3 -> 68.5 mm, vias 36 -> 22
- net /VDD3V3: track 19.8 -> 19.7 mm, vias 66 -> 62
- net /S2: vias 35 -> 21
- net /S1: vias 35 -> 21
- added copper zone on In1.Cu, net /S1
- added copper zone on In2.Cu, net /S1
- added copper zone on In1.Cu, net /S2
- added copper zone on In1.Cu, net /S3
- added copper zone on In2.Cu, net /S3
- added copper zone on In2.Cu, net GND

Commit message: LAYOUT
Routing:
- net (no net): vias 0 -> 3
Other:
- board size 71.1 x 40 mm -> 96.7 x 40 mm
- board text added: "Bologna Design"

Commit message: update
Parts:
- added CPIN1: GRJ31CZ72A475KE01L, SamacSys_Parts:CAPC3216X190N, F.Cu at (74.0, 85.6)
- added CPIN2: GRJ31CZ72A475KE01L, SamacSys_Parts:CAPC3216X190N, F.Cu at (74.0, 87.9)
- added TPC1: TestPoint, TestPoint:TestPoint_Pad_1.0x1.0mm, F.Cu at (77.9, 101.0)
- added TPG1: TestPoint, TestPoint:TestPoint_Pad_1.0x1.0mm, F.Cu at (67.2, 92.8)
- added TPG2: TestPoint, TestPoint:TestPoint_Pad_1.0x1.0mm, F.Cu at (67.4, 101.2)
- added TPG3: TestPoint, TestPoint:TestPoint_Pad_1.0x1.0mm, F.Cu at (67.4, 108.5)
- added TPG4: TestPoint, TestPoint:TestPoint_Pad_1.0x1.0mm, F.Cu at (67.1, 116.6)
- added TPGND1: TestPoint, TestPoint:TestPoint_Pad_1.0x1.0mm, F.Cu at (24.8, 118.1)
- added TPS1: TestPoint, TestPoint:TestPoint_Pad_1.0x1.0mm, F.Cu at (77.9, 96.3)
- added TPS3: TestPoint, TestPoint:TestPoint_Pad_1.0x1.0mm, F.Cu at (77.0, 110.0)
- COL1, COL2: value C -> GRM0335C1E5R1BA01D
- J1: value 62000211121_x6 -> Conn_01x05; footprint SamacSys_Parts:62000211121_x6 -> Connector_PinHeader_2.54mm:PinHeader_1x05_P2.54mm_Vertical
- J2: value 62000211121 -> Conn_01x02; footprint SamacSys_Parts:62000211121 -> Connector_PinHeader_2.54mm:PinHeader_1x02_P2.54mm_Vertical
- J3, J4: value 62000211121_x1 -> Conn_01x01; footprint SamacSys_Parts:62000211121_x1 -> Connector_PinHeader_2.54mm:PinHeader_1x01_P2.54mm_Vertical
- RS1, RS4, RS8: value R -> RT0603DRE10100KL
- RS2, RS3: value R -> RT0603DRE077K41L
- RS7: value R -> RP0603BRD075K76L
- moved P2 5.94 mm to (83.8, 82.8), turned to 180 degrees
- moved C3 5.16 mm to (82.2, 88.4), turned to 180 degrees
- moved J4 1.63 mm to (21.5, 117.4)
- moved J1 1.36 mm to (17.7, 97.2), turned to 0 degrees
- moved J2 1.36 mm to (17.7, 113.5), turned to 180 degrees
- moved J3 1.27 mm to (17.8, 117.4)
Routing:
- net /S2: track 150.9 -> 142.2 mm
- net GND: track 333.4 -> 336.7 mm, vias 232 -> 250
- net /NRST: track 41.2 -> 44.3 mm
- net /COMP2_INM: track 15.5 -> 17.8 mm
- net /T_SWDIO: track 24.8 -> 26.7 mm
- net /STLINK_RX: track 18.2 -> 19.7 mm
- net /STLINK_TX: track 15.6 -> 17.0 mm
- net /T_SWCLK: track 22.7 -> 23.9 mm
- net /COMP1_INM: track 18.5 -> 19.7 mm

Commit message: modded
Parts:
- removed TPGND1: TestPoint, TestPoint:TestPoint_Pad_1.0x1.0mm
- added J5: Conn_01x01, Connector_PinHeader_2.54mm:PinHeader_1x01_P2.54mm_Vertical, F.Cu at (25.2, 117.4)
- moved RS2 1.29 mm to (29.9, 117.4)
- moved RS3 1.27 mm to (37.1, 118.4)
- moved Z1 1.24 mm to (29.6, 115.1)
- moved Z2 1.24 mm to (37.2, 116.1)
- moved RS1 1.06 mm to (32.3, 116.6)
- moved RS4 0.88 mm to (33.9, 116.6)
Routing:
- net GND: track 336.7 -> 329.7 mm
- net /COMP1_INP: track 25.6 -> 24.0 mm
- net /S2: track 142.2 -> 141.2 mm
- net /ADC1_IN1: track 18.9 -> 18.1 mm
