File: MuReSC_GaN_v1/Project.kicad_sch (KiCad schematic)
At the start: 115 parts, among them IC1 STM32G474RET6, IC10 UCC12040DVE, IC11 LMG1020YFFR, IC12 LMG1020YFFR, IC13 LMG1020YFFR, IC14 LMG1020YFFR, IC2 TPSM5601R5HRDAR, IC3 ISO7720FQDQ1, IC4 ISO7720FQDQ1, IC5 ISO7720FQDQ1, IC6 ISO7720FQDQ1, IC7 UCC12040DVE, IC8 UCC12040DVE, IC9 UCC12040DVE, J1 62000211121_x6, J2 62000211121, J3 62000211121_x1, J4 62000211121_x1, P1 691214110002, P2 691214110002, Q1 GS61004B-TR, Q2 GS61004B-TR, Q3 GS61004B-TR, Q4 GS61004B-TR, Y1 NX3215SA-32.768K-STD-MUS-2, Y2 NX3225SA-24.000MHZ-STD-CSR-1

Commit message: quasi finito
Parts:
- removed RS5, RS6: R, Resistor_SMD:R_0603_1608Metric_Pad0.98x0.95mm_HandSolder, symbol Device:R
- removed Z4: TSZU52C3V3_RGG, TSZU52C3V3RGG, symbol SamacSys_Parts:TSZU52C3V3_RGG
Connections:
- net COMP2_INP is gone; now on net ADC2_IN2: IC1.21 (PA7)
- net CENTER: now reaches C1.2, C2.1, L1.1
Changed lines of the file:
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@@
   (junction (at 326.39 250.19) (diameter 0) (color 0 0 0 0)
   )
-  (junction (at 477.52 36.83) (diameter 0) (color 0 0 0 0)
-  )
   (junction (at 274.32 107.95) (diameter 0) (color 0 0 0 0)
   )
@@
   (junction (at 326.39 245.11) (diameter 0) (color 0 0 0 0)
   )
-  (junction (at 477.52 52.07) (diameter 0) (color 0 0 0 0)
-  )
   (junction (at 328.93 179.07) (diameter 0) (color 0 0 0 0)
   )
@@
     (stroke (width 0) (type default))
   )
-  (wire (pts (xy 477.52 22.86) (xy 477.52 26.67))
-    (stroke (width 0) (type default))
-  )
   (wire (pts (xy 265.43 232.41) (xy 271.78 232.41))
     (stroke (width 0) (type default))
@@
     (stroke (width 0) (type default))
   )
-  (wire (pts (xy 490.22 36.83) (xy 477.52 36.83))
-    (stroke (width 0) (type default))
-  )
   (wire (pts (xy 21.59 200.66) (xy 29.21 200.66))
     (stroke (width 0) (type default))
@@
     (stroke (width 0) (type default))
   )
-  (wire (pts (xy 477.52 36.83) (xy 477.52 40.64))
-    (stroke (width 0) (type default))
-  )
   (wire (pts (xy 407.67 175.26) (xy 414.02 175.26))
     (stroke (width 0) (type default))
@@
     (stroke (width 0) (type default))
   )
-  (wire (pts (xy 477.52 34.29) (xy 477.52 36.83))
-    (stroke (width 0) (type default))
-  )
   (wire (pts (xy 318.77 133.35) (xy 320.04 133.35))
     (stroke (width 0) (type default))
@@
     (stroke (width 0) (type default))
   )
-  (wire (pts (xy 477.52 52.07) (xy 477.52 48.26))
-    (stroke (width 0) (type default))
-  )
   (wire (pts (xy 560.07 212.09) (xy 560.07 273.05))
     (stroke (width 0) (type default))
@@
     (stroke (width 0) (type default))
   )
-  (wire (pts (xy 477.52 52.07) (xy 477.52 53.34))
-    (stroke (width 0) (type default))
-  )
   (wire (pts (xy 506.73 99.06) (xy 506.73 109.22))
     (stroke (width 0) (type default))
@@
     (stroke (width 0) (type default))
   )
-  (wire (pts (xy 490.22 52.07) (xy 477.52 52.07))
-    (stroke (width 0) (type default))
-  )
   (wire (pts (xy 326.39 326.39) (xy 326.39 328.93))
     (stroke (width 0) (type default))
@@
     (effects (font (size 1.27 1.27)) (justify left bottom))
   )
-  (label "COMP2_INP" (at 478.79 36.83 0) (fields_autoplaced)
-    (effects (font (size 1.27 1.27)) (justify left bottom))
-  )
   (label "S2" (at 326.39 166.37 0) (fields_autoplaced)
     (effects (font (size 1.27 1.27)) (justify left bottom))
@@
     (effects (font (size 1.27 1.27)) (justify left bottom))
   )
+  (label "COMP2_INP" (at 443.23 38.1 0) (fields_autoplaced)
+    (effects (font (size 1.27 1.27)) (justify left bottom))
+  )
   (label "VDD48V" (at 279.4 25.4 0) (fields_autoplaced)
     (effects (font (size 1.27 1.27)) (justify left bottom))
@@
     (effects (font (size 1.27 1.27)) (justify left bottom))
   )
-  (label "VDD48V" (at 477.52 22.86 0) (fields_autoplaced)
-    (effects (font (size 1.27 1.27)) (justify left bottom))
-  )
   (label "VDDI2" (at 379.73 175.26 0) (fields_autoplaced)
     (effects (font (size 1.27 1.27)) (justify left bottom))
@@
     (effects (font (size 1.27 1.27)) (justify left bottom))
   )
+  (label "CENTER" (at 560.07 182.88 0) (fields_autoplaced)
+    (effects (font (size 1.27 1.27)) (justify left bottom))
+  )
   (label "INP1" (at 224.79 121.92 0) (fields_autoplaced)
     (effects (font (size 1.27 1.27)) (justify left bottom))
@@
     )
   )
-  (symbol (lib_id "Device:R") (at 477.52 30.48 0) (unit 1)
-    (in_bom yes) (on_board yes) (dnp no) (fields_autoplaced)
-    (property "Reference" "RS5" (at 480.06 29.21 0)
-      (effects (font (size 1.27 1.27)) (justify left))
-    )
-    (property "Value" "R" (at 480.06 31.75 0)
-      (effects (font (size 1.27 1.27)) (justify left))
-    )
-    (property "Footprint" "Resistor_SMD:R_0603_1608Metric_Pad0.98x0.95mm_HandSolder" (at 475.742 30.48 90)
-      (effects (font (size 1.27 1.27)) hide)
-    )
-    (property "Datasheet" "~" (at 477.52 30.48 0)
-      (effects (font (size 1.27 1.27)) hide)
-    )
-    (pin "1")
-    (pin "2")
-    (instances
-      (project "Project"
-        (path "/370b4fcc-a080-452a-8e5f-5eff99707865"
-          (reference "RS5") (unit 1)
-        )
-      )
-    )
-  )
   (symbol (lib_id "SamacSys_Parts:GRT155R70J105KE01D") (at 228.6 318.77 270) (unit 1)
     (in_bom yes) (on_board yes) (dnp no)
@@
     )
   )
-  (symbol (lib_id "SamacSys_Parts:TSZU52C3V3_RGG") (at 490.22 36.83 270) (unit 1)
-    (in_bom yes) (on_board yes) (dnp no) (fields_autoplaced)
-    (property "Reference" "Z4" (at 494.03 43.18 90)
-      (effects (font (size 1.27 1.27)) (justify left))
-    )
-    (property "Value" "TSZU52C3V3_RGG" (at 494.03 45.72 90)
-      (effects (font (size 1.27 1.27)) (justify left))
-    )
-    (property "Footprint" "TSZU52C3V3RGG" (at 396.57 46.99 0)
-      (effects (font (size 1.27 1.27)) (justify left top) hide)
-    )
-    (property "Datasheet" "https://www.taiwansemi.com/assets/uploads/datasheet/TSZU52C2V0%20SERIES_G2009.pdf" (at 296.57 46.99 0)
-      (effects (font (size 1.27 1.27)) (justify left top) hide)
-    )
-    (property "Height" "0.85" (at 96.57 46.99 0)
-      (effects (font (size 1.27 1.27)) (justify left top) hide)
-    )
-    (property "Mouser Part Number" "821-TSZU52C3V3RGG" (at -3.43 46.99 0)
-      (effects (font (size 1.27 1.27)) (justify left top) hide)
-    )
-    (property "Mouser Price/Stock" "https://www.mouser.co.uk/ProductDetail/Taiwan-Semiconductor/TSZU52C3V3-RGG?qs=QEzMiVqgwc2LOQHSCGq8kg%3D%3D" (at -103.43 46.99 0)
-      (effects (font (size 1.27 1.27)) (justify left top) hide)
-    )
-    (property "Manufacturer_Name" "Taiwan Semiconductor" (at -203.43 46.99 0)
-      (effects (font (size 1.27 1.27)) (justify left top) hide)
-    )
-    (property "Manufacturer_Part_Number" "TSZU52C3V3 RGG" (at -303.43 46.99 0)
-      (effects (font (size 1.27 1.27)) (justify left top) hide)
-    )
-    (pin "1")
-    (pin "2")
-    (instances
-      (project "Project"
-        (path "/370b4fcc-a080-452a-8e5f-5eff99707865"
-          (reference "Z4") (unit 1)
-        )
-      )
-    )
-  )
   (symbol (lib_id "power:GND") (at 25.4 231.14 270) (unit 1)
     (in_bom yes) (on_board yes) (dnp no) (fields_autoplaced)
@@
     )
   )
-  (symbol (lib_id "power:GND") (at 477.52 53.34 0) (unit 1)
-    (in_bom yes) (on_board yes) (dnp no) (fields_autoplaced)
-    (property "Reference" "#PWR016" (at 477.52 59.69 0)
-      (effects (font (size 1.27 1.27)) hide)
-    )
-    (property "Value" "GND" (at 477.52 58.42 0)
-      (effects (font (size 1.27 1.27)))
-    )
-    (property "Footprint" "" (at 477.52 53.34 0)
-      (effects (font (size 1.27 1.27)) hide)
-    )
-    (property "Datasheet" "" (at 477.52 53.34 0)
-      (effects (font (size 1.27 1.27)) hide)
-    )
-    (pin "1")
-    (instances
-      (project "Project"
-        (path "/370b4fcc-a080-452a-8e5f-5eff99707865"
-          (reference "#PWR016") (unit 1)
-        )
-      )
-    )
-  )
   (symbol (lib_id "SamacSys_Parts:C0402C104K8RAC7867") (at 265.43 300.99 270) (unit 1)
     (in_bom yes) (on_board yes) (dnp no) (fields_autoplaced)
@@
         )
       )
-    )
-  )
-  (symbol (lib_id "Device:R") (at 477.52 44.45 0) (unit 1)
-    (in_bom yes) (on_board yes) (dnp no) (fields_autoplaced)
-    (property "Reference" "RS6" (at 480.06 43.18 0)
-      (effects (font (size 1.27 1.27)) (justify left))
-    )
-    (property "Value" "R" (at 480.06 45.72 0)
-      (effects (font (size 1.27 1.27)) (justify left))
-    )
-    (property "Footprint" "Resistor_SMD:R_0603_1608Metric_Pad0.98x0.95mm_HandSolder" (at 475.742 44.45 90)
-      (effects (font (size 1.27 1.27)) hide)
-    )
-    (property "Datasheet" "~" (at 477.52 44.45 0)
-      (effects (font (size 1.27 1.27)) hide)
-    )
-    (pin "1")
-    (pin "2")
-    (instances
-      (project "Project"
-        (path "/370b4fcc-a080-452a-8e5f-5eff99707865"
-          (reference "RS6") (unit 1)
-        )
-      )

Commit message: LAYOUT DRC
Parts:
- COH1: footprint CAPC0603X33N -> SamacSys_Parts:CAPC0603X33N
- COL1, COL2: footprint Capacitor_SMD:C_0201_0603Metric_Pad0.64x0.40mm_HandSolder -> SamacSys_Parts:CAPC0603X33N
Changed lines of the file:
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@@
       (effects (font (size 1.27 1.27)))
     )
-    (property "Footprint" "Capacitor_SMD:C_0201_0603Metric_Pad0.64x0.40mm_HandSolder" (at 36.83 199.6948 0)
+    (property "Footprint" "SamacSys_Parts:CAPC0603X33N" (at 36.83 199.6948 0)
       (effects (font (size 1.27 1.27)) hide)
     )
@@
       (effects (font (size 1.27 1.27)))
     )
-    (property "Footprint" "CAPC0603X33N" (at 36.83 327.33 0)
+    (property "Footprint" "SamacSys_Parts:CAPC0603X33N" (at 36.83 327.33 0)
       (effects (font (size 1.27 1.27)) (justify left top) hide)
     )
@@
       (effects (font (size 1.27 1.27)))
     )
-    (property "Footprint" "Capacitor_SMD:C_0201_0603Metric_Pad0.64x0.40mm_HandSolder" (at 36.83 213.6648 0)
+    (property "Footprint" "SamacSys_Parts:CAPC0603X33N" (at 36.83 213.6648 0)
       (effects (font (size 1.27 1.27)) hide)
     )

Commit message: update
Parts:
- removed J1: 62000211121_x6, SamacSys_Parts:62000211121_x6, symbol SamacSys_Parts:62000211121_x6
- removed J2: 62000211121, 62000211121, symbol SamacSys_Parts:62000211121
- removed J3, J4: 62000211121_x1, SamacSys_Parts:62000211121_x1, symbol SamacSys_Parts:62000211121_x1
- added CPIN1, CPIN2: GRJ31CZ72A475KE01L, CAPC3216X190N, symbol SamacSys_Parts:GRJ31CZ72A475KE01L
- added J1: Conn_01x05, Connector_PinHeader_2.54mm:PinHeader_1x05_P2.54mm_Vertical, symbol Connector_Generic:Conn_01x05
- added J2: Conn_01x02, Connector_PinHeader_2.54mm:PinHeader_1x02_P2.54mm_Vertical, symbol Connector_Generic:Conn_01x02
- added J3, J4: Conn_01x01, Connector_PinHeader_2.54mm:PinHeader_1x01_P2.54mm_Vertical, symbol Connector_Generic:Conn_01x01
- added TPC1, TPG1, TPG2, TPG3, TPG4, TPGND1, TPS1, TPS3: TestPoint, TestPoint:TestPoint_Pad_1.0x1.0mm, symbol Connector:TestPoint
- COL1, COL2: value C -> GRM0335C1E5R1BA01D
- RS1, RS4, RS8: value R -> RT0603DRE10100KL
- RS2, RS3: value R -> RT0603DRE077K41L
- RS7: value R -> RP0603BRD075K76L
Connections:
- net CENTER: now also TPC1.1
- net COMP1_INM: now also J3.1 (Pin_1)
- net COMP2_INM: now also J4.1 (Pin_1)
- net G1: now also TPG1.1
- net G2: now also TPG2.1
- net G3: now also TPG3.1
- net G4: now also TPG4.1
- net GND: now also CPIN1.2, CPIN2.2, J1.3 (Pin_3), TPGND1.1
- net NRST: now also J1.5 (Pin_5)
- net S1: now also TPS1.1
- net S3: now also TPS3.1
- net STLINK_RX: now also J2.2 (Pin_2)
- net STLINK_TX: now also J2.1 (Pin_1)
- net T_SWCLK: now also J1.2 (Pin_2)
- net T_SWDIO: now also J1.4 (Pin_4)
- net VDD3V3: now also J1.1 (Pin_1)
- net VDD48V: now also CPIN1.1, CPIN2.1
Other:
- note removed: "CAPACITA FILRO QUI?"

Commit message: modded
Parts:
- removed TPGND1: TestPoint, TestPoint:TestPoint_Pad_1.0x1.0mm, symbol Connector:TestPoint
- added J5: Conn_01x01, Connector_PinHeader_2.54mm:PinHeader_1x01_P2.54mm_Vertical, symbol Connector_Generic:Conn_01x01
Connections:
- net GND: now also J5.1 (Pin_1)
Changed lines of the file:
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@@
     )
   )
+  (symbol (lib_id "Connector_Generic:Conn_01x01") (at 332.74 62.23 0) (unit 1)
+    (in_bom yes) (on_board yes) (dnp no) (fields_autoplaced)
+    (property "Reference" "J5" (at 335.28 60.96 0)
+      (effects (font (size 1.27 1.27)) (justify left))
+    )
+    (property "Value" "Conn_01x01" (at 335.28 63.5 0)
+      (effects (font (size 1.27 1.27)) (justify left))
+    )
+    (property "Footprint" "Connector_PinHeader_2.54mm:PinHeader_1x01_P2.54mm_Vertical" (at 332.74 62.23 0)
+      (effects (font (size 1.27 1.27)) hide)
+    )
+    (property "Datasheet" "~" (at 332.74 62.23 0)
+      (effects (font (size 1.27 1.27)) hide)
+    )
+    (pin "1")
+    (instances
+      (project "Project"
+        (path "/370b4fcc-a080-452a-8e5f-5eff99707865"
+          (reference "J5") (unit 1)
+        )
+      )
+    )
+  )
   (symbol (lib_id "Connector:TestPoint") (at 490.22 234.95 270) (unit 1)
     (in_bom yes) (on_board yes) (dnp no) (fields_autoplaced)
@@
         )
       )
-    )
-  )
-  (symbol (lib_id "Connector:TestPoint") (at 327.66 62.23 270) (unit 1)
-    (in_bom yes) (on_board yes) (dnp no) (fields_autoplaced)
-    (property "Reference" "TPGND1" (at 332.74 60.96 90)
-      (effects (font (size 1.27 1.27)) (justify left))
-    )
-    (property "Value" "TestPoint" (at 332.74 63.5 90)
-      (effects (font (size 1.27 1.27)) (justify left))
-    )
-    (property "Footprint" "TestPoint:TestPoint_Pad_1.0x1.0mm" (at 327.66 67.31 0)
-      (effects (font (size 1.27 1.27)) hide)
-    )
-    (property "Datasheet" "~" (at 327.66 67.31 0)
-      (effects (font (size 1.27 1.27)) hide)
-    )
-    (pin "1")
-    (instances
-      (project "Project"
-        (path "/370b4fcc-a080-452a-8e5f-5eff99707865"
-          (reference "TPGND1") (unit 1)
-        )
-      )
