File: MuReSC_GaN_v1/Project.kicad_sch (KiCad schematic)
At the start: 122 parts, among them IC1 STM32G474RET6, IC10 UCC12040DVE, IC11 LMG1020YFFR, IC12 LMG1020YFFR, IC13 LMG1020YFFR, IC14 LMG1020YFFR, IC2 TPSM5601R5HRDAR, IC3 ISO7720FQDQ1, IC4 ISO7720FQDQ1, IC5 ISO7720FQDQ1, IC6 ISO7720FQDQ1, IC7 UCC12040DVE, IC8 UCC12040DVE, IC9 UCC12040DVE, J1 Conn_01x05, J2 Conn_01x02, J3 Conn_01x01, J4 Conn_01x01, J5 Conn_01x01, P1 691214110002, P2 691214110002, Q1 GS61004B-TR, Q2 GS61004B-TR, Q3 GS61004B-TR, Q4 GS61004B-TR, Y1 NX3215SA-32.768K-STD-MUS-2, Y2 NX3225SA-24.000MHZ-STD-CSR-1

Commit message: update
Parts:
- added JP1: Jumper_2_Bridged, Connector_PinHeader_2.54mm:PinHeader_1x02_P2.54mm_Vertical, symbol Jumper:Jumper_2_Bridged
Connections:
- net VDD48V: now also JP1.1 (A), JP1.2 (B)
Changed lines of the file:
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@@
     (stroke (width 0) (type default))
   )
+  (wire (pts (xy 276.86 62.23) (xy 288.29 62.23))
+    (stroke (width 0) (type default))
+  )
   (wire (pts (xy 490.22 109.22) (xy 490.22 110.49))
     (stroke (width 0) (type default))
@@
     (stroke (width 0) (type default))
   )
+  (wire (pts (xy 298.45 62.23) (xy 306.07 62.23))
+    (stroke (width 0) (type default))
+  )
   (wire (pts (xy 17.78 121.92) (xy 20.32 121.92))
     (stroke (width 0) (type default))
@@
     (effects (font (size 1.27 1.27)) (justify left bottom))
   )
+  (label "VDD48V" (at 306.07 62.23 0) (fields_autoplaced)
+    (effects (font (size 1.27 1.27)) (justify left bottom))
+  )
   (label "VDD3V3" (at 186.69 241.3 0) (fields_autoplaced)
     (effects (font (size 1.27 1.27)) (justify left bottom))
@@
     (effects (font (size 1.27 1.27)) (justify left bottom))
   )
+  (label "VDD48V" (at 276.86 62.23 0) (fields_autoplaced)
+    (effects (font (size 1.27 1.27)) (justify left bottom))
+  )
   (label "VDD3V3" (at 93.98 143.51 90) (fields_autoplaced)
     (effects (font (size 1.27 1.27)) (justify left bottom))
@@
         )
       )
+    )
+  )
+  (symbol (lib_id "Jumper:Jumper_2_Bridged") (at 293.37 62.23 0) (unit 1)
+    (in_bom yes) (on_board yes) (dnp no) (fields_autoplaced)
+    (property "Reference" "JP1" (at 293.37 57.15 0)
+      (effects (font (size 1.27 1.27)))
+    )
+    (property "Value" "Jumper_2_Bridged" (at 293.37 59.69 0)
+      (effects (font (size 1.27 1.27)))
+    )
+    (property "Footprint" "Connector_PinHeader_2.54mm:PinHeader_1x02_P2.54mm_Vertical" (at 293.37 62.23 0)
+      (effects (font (size 1.27 1.27)) hide)
+    )
+    (property "Datasheet" "~" (at 293.37 62.23 0)
+      (effects (font (size 1.27 1.27)) hide)
+    )
+    (pin "1")
+    (pin "2")
+    (instances
+      (project "Project"
+        (path "/370b4fcc-a080-452a-8e5f-5eff99707865"
+          (reference "JP1") (unit 1)
+        )
+      )

Commit message: footprint
Parts:
- CISOP1, CISOP2, CISOP3, CISOP4, CISOS1, CISOS2, CISOS3, CISOS4: value GRT155R70J105KE01D -> C0402C104K8RACTU
- CM1, CM10, CM2, CM3, CM4, CM6, CM7, CM9, CTP1, CTP2, CTP3, CTP4, CTS1, CTS2, CTS3, CTS4: value C0402C104K8RAC7867 -> C0402C104K8RACTU
- J1: footprint Connector_PinHeader_2.54mm:PinHeader_1x05_P2.54mm_Vertical -> SamacSys_Parts:PinHeader_1x05_P2.54mm_Horizontal
- J2, JP1: footprint Connector_PinHeader_2.54mm:PinHeader_1x02_P2.54mm_Vertical -> SamacSys_Parts:PinHeader_1x02_P2.54mm_Horizontal
Changed lines of the file:
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@@
       (effects (font (size 1.27 1.27)) (justify left))
     )
-    (property "Value" "GRT155R70J105KE01D" (at 232.41 187.96 90)
+    (property "Value" "C0402C104K8RACTU" (at 232.41 187.96 90)
       (effects (font (size 1.27 1.27)) (justify left))
     )
@@
       (effects (font (size 1.27 1.27)) (justify left))
     )
-    (property "Value" "C0402C104K8RAC7867" (at 271.78 158.75 90)
+    (property "Value" "C0402C104K8RACTU" (at 271.78 158.75 90)
       (effects (font (size 1.27 1.27)) (justify left))
     )
@@
       (effects (font (size 1.27 1.27)) (justify right))
     )
-    (property "Value" "C0402C104K8RAC7867" (at 63.5 176.53 90)
+    (property "Value" "C0402C104K8RACTU" (at 63.5 176.53 90)
       (effects (font (size 1.27 1.27)) (justify right))
     )
@@
       (effects (font (size 1.27 1.27)) (justify left))
     )
-    (property "Value" "GRT155R70J105KE01D" (at 228.6 327.66 90)
+    (property "Value" "C0402C104K8RACTU" (at 228.6 327.66 90)
       (effects (font (size 1.27 1.27)) (justify left))
     )
@@
       (effects (font (size 1.27 1.27)) (justify left))
     )
-    (property "Value" "GRT155R70J105KE01D" (at 231.14 247.65 90)
+    (property "Value" "C0402C104K8RACTU" (at 231.14 247.65 90)
       (effects (font (size 1.27 1.27)) (justify left))
     )
@@
       (effects (font (size 1.27 1.27)) (justify left))
     )
-    (property "Value" "C0402C104K8RAC7867" (at 323.85 308.61 90)
+    (property "Value" "C0402C104K8RACTU" (at 323.85 308.61 90)
       (effects (font (size 1.27 1.27)) (justify left))
     )
@@
       (effects (font (size 1.27 1.27)))
     )
-    (property "Value" "C0402C104K8RAC7867" (at 104.14 138.43 0)
+    (property "Value" "C0402C104K8RACTU" (at 104.14 138.43 0)
       (effects (font (size 1.27 1.27)))
     )
@@
       (effects (font (size 1.27 1.27)) (justify left))
     )
-    (property "Value" "C0402C104K8RAC7867" (at 16.51 276.86 90)
+    (property "Value" "C0402C104K8RACTU" (at 16.51 276.86 90)
       (effects (font (size 1.27 1.27)) (justify left))
     )
@@
       (effects (font (size 1.27 1.27)))
     )
-    (property "Footprint" "Connector_PinHeader_2.54mm:PinHeader_1x02_P2.54mm_Vertical" (at 293.37 62.23 0)
+    (property "Footprint" "SamacSys_Parts:PinHeader_1x02_P2.54mm_Horizontal" (at 293.37 62.23 0)
       (effects (font (size 1.27 1.27)) hide)
     )
@@
       (effects (font (size 1.27 1.27)) (justify left))
     )
-    (property "Value" "C0402C104K8RAC7867" (at 41.91 341.63 90)
+    (property "Value" "C0402C104K8RACTU" (at 41.91 341.63 90)
       (effects (font (size 1.27 1.27)) (justify left))
     )
@@
       (effects (font (size 1.27 1.27)) (justify left))
     )
-    (property "Value" "C0402C104K8RAC7867" (at 271.78 100.33 90)
+    (property "Value" "C0402C104K8RACTU" (at 271.78 100.33 90)
       (effects (font (size 1.27 1.27)) (justify left))
     )
@@
       (effects (font (size 1.27 1.27)) (justify left))
     )
-    (property "Value" "GRT155R70J105KE01D" (at 232.41 125.73 90)
+    (property "Value" "C0402C104K8RACTU" (at 232.41 125.73 90)
       (effects (font (size 1.27 1.27)) (justify left))
     )
@@
       (effects (font (size 1.27 1.27)) (justify left))
     )
-    (property "Value" "C0402C104K8RAC7867" (at 326.39 158.75 90)
+    (property "Value" "C0402C104K8RACTU" (at 326.39 158.75 90)
       (effects (font (size 1.27 1.27)) (justify left))
     )
@@
       (effects (font (size 1.27 1.27)) (justify left))
     )
-    (property "Value" "C0402C104K8RAC7867" (at 326.39 100.33 90)
+    (property "Value" "C0402C104K8RACTU" (at 326.39 100.33 90)
       (effects (font (size 1.27 1.27)) (justify left))
     )
@@
       (effects (font (size 1.27 1.27)) (justify left))
     )
-    (property "Value" "GRT155R70J105KE01D" (at 190.5 237.49 0)
+    (property "Value" "C0402C104K8RACTU" (at 190.5 237.49 0)
       (effects (font (size 1.27 1.27)) (justify left))
     )
@@
       (effects (font (size 1.27 1.27)) (justify left))
     )
-    (property "Value" "C0402C104K8RAC7867" (at 269.24 308.61 90)
+    (property "Value" "C0402C104K8RACTU" (at 269.24 308.61 90)
       (effects (font (size 1.27 1.27)) (justify left))
     )
@@
       (effects (font (size 1.27 1.27)) (justify right))
     )
-    (property "Value" "C0402C104K8RAC7867" (at 95.25 176.53 90)
+    (property "Value" "C0402C104K8RACTU" (at 95.25 176.53 90)
       (effects (font (size 1.27 1.27)) (justify right))
     )
@@
       (effects (font (size 1.27 1.27)) (justify left))
     )
-    (property "Value" "C0402C104K8RAC7867" (at 323.85 224.79 90)
+    (property "Value" "C0402C104K8RACTU" (at 323.85 224.79 90)
       (effects (font (size 1.27 1.27)) (justify left))
     )
@@
       (effects (font (size 1.27 1.27)) (justify left))
     )
-    (property "Footprint" "Connector_PinHeader_2.54mm:PinHeader_1x05_P2.54mm_Vertical" (at 288.29 49.53 0)
+    (property "Footprint" "SamacSys_Parts:PinHeader_1x05_P2.54mm_Horizontal" (at 288.29 49.53 0)
       (effects (font (size 1.27 1.27)) hide)
     )
@@
       (effects (font (size 1.27 1.27)))
     )
-    (property "Value" "C0402C104K8RAC7867" (at 130.81 86.36 0)
+    (property "Value" "C0402C104K8RACTU" (at 130.81 86.36 0)
       (effects (font (size 1.27 1.27)))
     )
@@
       (effects (font (size 1.27 1.27)) (justify left))
     )
-    (property "Footprint" "Connector_PinHeader_2.54mm:PinHeader_1x02_P2.54mm_Vertical" (at 332.74 40.64 0)
+    (property "Footprint" "SamacSys_Parts:PinHeader_1x02_P2.54mm_Horizontal" (at 332.74 40.64 0)
       (effects (font (size 1.27 1.27)) hide)
     )
@@
       (effects (font (size 1.27 1.27)) (justify left))
     )
-    (property "Value" "GRT155R70J105KE01D" (at 187.96 317.5 0)
+    (property "Value" "C0402C104K8RACTU" (at 187.96 317.5 0)
       (effects (font (size 1.27 1.27)) (justify left))
     )
@@
       (effects (font (size 1.27 1.27)) (justify left))
     )
-    (property "Value" "C0402C104K8RAC7867" (at 269.24 224.79 90)
+    (property "Value" "C0402C104K8RACTU" (at 269.24 224.79 90)
       (effects (font (size 1.27 1.27)) (justify left))
     )
@@
       (effects (font (size 1.27 1.27)) (justify left))
     )
-    (property "Value" "GRT155R70J105KE01D" (at 193.04 177.8 0)
+    (property "Value" "C0402C104K8RACTU" (at 193.04 177.8 0)
       (effects (font (size 1.27 1.27)) (justify left))
     )
@@
       (effects (font (size 1.27 1.27)) (justify left))
     )
-    (property "Value" "GRT155R70J105KE01D" (at 193.04 115.57 0)
+    (property "Value" "C0402C104K8RACTU" (at 193.04 115.57 0)
       (effects (font (size 1.27 1.27)) (justify left))
     )
@@
       (effects (font (size 1.27 1.27)) (justify left))
     )
-    (property "Value" "C0402C104K8RAC7867" (at 20.32 130.81 90)
+    (property "Value" "C0402C104K8RACTU" (at 20.32 130.81 90)
       (effects (font (size 1.27 1.27)) (justify left))
     )
@@
       (effects (font (size 1.27 1.27)))
     )
-    (property "Value" "C0402C104K8RAC7867" (at 45.72 71.12 0)
+    (property "Value" "C0402C104K8RACTU" (at 45.72 71.12 0)
       (effects (font (size 1.27 1.27)))
     )

Commit message: up
Connections:
- net VDD3V3: now also BEAD1.1, CM1.1
Changed lines of the file:
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@@
     (effects (font (size 1.27 1.27)) (justify left bottom))
+  )
+  (label "VDD3V3" (at 19.05 121.92 180) (fields_autoplaced)
+    (effects (font (size 1.27 1.27)) (justify right bottom))
   )
   (label "S1" (at 326.39 107.95 0) (fields_autoplaced)
