File: MuReSC_BCD_v1/MuReSC_BCD.kicad_pcb (KiCad board)
At the start: 4 copper layers, 0 parts

Commit message: up
Parts:
- added C1: 100 nF, Capacitor_SMD:C_0603_1608Metric_Pad1.08x0.95mm_HandSolder, F.Cu at (155.1, 91.8)
- added C10: 1µF, Capacitor_SMD:C_0603_1608Metric_Pad1.08x0.95mm_HandSolder, F.Cu at (88.8, 152.7)
- added C11: 1µF, Capacitor_SMD:C_0603_1608Metric_Pad1.08x0.95mm_HandSolder, F.Cu at (88.8, 155.2)
- added C12: 100 nF, Capacitor_SMD:C_0603_1608Metric_Pad1.08x0.95mm_HandSolder, F.Cu at (88.8, 157.7)
- added C13: 1µF, Capacitor_SMD:C_0603_1608Metric_Pad1.08x0.95mm_HandSolder, F.Cu at (88.8, 160.2)
- added C14: 10 nF, Capacitor_SMD:C_0603_1608Metric_Pad1.08x0.95mm_HandSolder, F.Cu at (88.8, 162.8)
- added C15: 10 uF, Capacitor_SMD:C_0603_1608Metric_Pad1.08x0.95mm_HandSolder, F.Cu at (88.8, 165.3)
- added C16: C, Capacitor_SMD:C_0603_1608Metric_Pad1.08x0.95mm_HandSolder, F.Cu at (88.8, 167.8)
- added C2: 1µF, Capacitor_SMD:C_0603_1608Metric_Pad1.08x0.95mm_HandSolder, F.Cu at (155.1, 93.5)
- added C3: 100n, Capacitor_SMD:C_0603_1608Metric_Pad1.08x0.95mm_HandSolder, F.Cu at (155.1, 95.2)
- added C4: 100n, Capacitor_SMD:C_0603_1608Metric_Pad1.08x0.95mm_HandSolder, F.Cu at (155.1, 97.0)
- added C5: 100n, Capacitor_SMD:C_0603_1608Metric_Pad1.08x0.95mm_HandSolder, F.Cu at (155.1, 98.8)
- added C6: 100n, Capacitor_SMD:C_0603_1608Metric_Pad1.08x0.95mm_HandSolder, F.Cu at (155.1, 100.5)
- added C7: 100n, Capacitor_SMD:C_0603_1608Metric_Pad1.08x0.95mm_HandSolder, F.Cu at (155.1, 102.2)
- added C8: 100 nF, Capacitor_SMD:C_0603_1608Metric_Pad1.08x0.95mm_HandSolder, F.Cu at (88.8, 147.7)
- added C9: 1µF, Capacitor_SMD:C_0603_1608Metric_Pad1.08x0.95mm_HandSolder, F.Cu at (75.1, 156.2)
- added CLAMP1: 691214110002, SamacSys_Parts:691214110002, F.Cu at (72.8, 99.8)
- added CLAMP2: 691214110002, SamacSys_Parts:691214110002, F.Cu at (72.2, 106.0)
- added CLAMP3: 691214110002, SamacSys_Parts:691214110002, F.Cu at (139.8, 122.8)
- added CMR1: C, Capacitor_SMD:C_0603_1608Metric_Pad1.08x0.95mm_HandSolder, F.Cu at (93.2, 147.7)
- added CMaR1: C, Capacitor_SMD:C_0603_1608Metric_Pad1.08x0.95mm_HandSolder, F.Cu at (93.2, 150.2)
- added COUT1: 100nF, Capacitor_SMD:C_0603_1608Metric_Pad1.08x0.95mm_HandSolder, F.Cu at (93.2, 152.7)
- added COUT2: 1µF, Capacitor_SMD:C_0603_1608Metric_Pad1.08x0.95mm_HandSolder, F.Cu at (93.2, 155.2)
- added COUT3: 10µF, Capacitor_SMD:C_0603_1608Metric_Pad1.08x0.95mm_HandSolder, F.Cu at (93.2, 157.7)
- added J1: Conn_Coaxial:60312002114503, Connector_Coaxial:SMA_Wurth_60312002114503_Vertical, F.Cu at (85.0, 72.8)
- added J10: Conn_Coaxial:60312002114503, Connector_Coaxial:SMA_Wurth_60312002114503_Vertical, F.Cu at (130.3, 72.9)
- added J11: Conn_Coaxial:60312002114503, Connector_Coaxial:SMA_Wurth_60312002114503_Vertical, F.Cu at (121.3, 125.2)
- added J12: Conn_Coaxial:60312002114503, Connector_Coaxial:SMA_Wurth_60312002114503_Vertical, F.Cu at (130.3, 107.6)
- added J13: Conn_Coaxial:60312002114503, Connector_Coaxial:SMA_Wurth_60312002114503_Vertical, F.Cu at (130.4, 98.9)
- added J14: Conn_Coaxial:60312002114503, Connector_Coaxial:SMA_Wurth_60312002114503_Vertical, F.Cu at (130.3, 125.0)
- added J2: Conn_Coaxial:60312002114503, Connector_Coaxial:SMA_Wurth_60312002114503_Vertical, F.Cu at (94.2, 72.8)
- added J3: Conn_Coaxial:60312002114503, Connector_Coaxial:SMA_Wurth_60312002114503_Vertical, F.Cu at (111.8, 72.8)
- added J4: Conn_Coaxial:60312002114503, Connector_Coaxial:SMA_Wurth_60312002114503_Vertical, F.Cu at (103.0, 72.8)
- added J5: Conn_Coaxial:60312002114503, Connector_Coaxial:SMA_Wurth_60312002114503_Vertical, F.Cu at (120.8, 72.8)
- added J6: Conn_01x04_Socket, Connector_PinHeader_2.54mm:PinHeader_1x04_P2.54mm_Vertical, F.Cu at (95.2, 81.0)
- added J7: Conn_Coaxial:60312002114503, Connector_Coaxial:SMA_Wurth_60312002114503_Vertical, F.Cu at (130.3, 81.6)
- added J8: Conn_Coaxial:60312002114503, Connector_Coaxial:SMA_Wurth_60312002114503_Vertical, F.Cu at (130.4, 90.4)
- added J9: Conn_Coaxial:60312002114503, Connector_Coaxial:SMA_Wurth_60312002114503_Vertical, F.Cu at (130.2, 116.2)
- added JP1: Jumper_3_Open, Connector_PinHeader_2.54mm:PinHeader_1x03_P2.54mm_Vertical, F.Cu at (83.2, 113.3)
- added JP2: Jumper_3_Open, Connector_PinHeader_2.54mm:PinHeader_1x03_P2.54mm_Vertical, F.Cu at (83.2, 108.7)
- added JP3: Jumper_3_Open, Connector_PinHeader_2.54mm:PinHeader_1x03_P2.54mm_Vertical, F.Cu at (83.2, 104.0)
- added JP4: Jumper_3_Open, Connector_PinHeader_2.54mm:PinHeader_1x03_P2.54mm_Vertical, F.Cu at (83.2, 99.4)
- added JP5: Jumper_3_Open, Connector_PinHeader_2.54mm:PinHeader_1x03_P2.54mm_Vertical, F.Cu at (83.2, 94.8)
- added JP6: Jumper_3_Open, Connector_PinHeader_2.54mm:PinHeader_1x03_P2.54mm_Vertical, F.Cu at (83.2, 90.1)
- added JP7: Jumper_3_Open, Connector_PinHeader_2.54mm:PinHeader_1x03_P2.54mm_Vertical, F.Cu at (83.2, 85.5)
- added JP8: Jumper_3_Open, Connector_PinHeader_2.54mm:PinHeader_1x03_P2.54mm_Vertical, F.Cu at (83.2, 80.8)
- added LR1: L, LCL:Coilcraft-Square-Air-Core-Inductors-all, F.Cu at (109.7, 107.8)
- added R1: 100k, Resistor_SMD:R_0603_1608Metric_Pad0.98x0.95mm_HandSolder, F.Cu at (93.2, 160.2)
- added R10: 100k, Resistor_SMD:R_0603_1608Metric_Pad0.98x0.95mm_HandSolder, F.Cu at (97.5, 160.2)
- added R11: 100k, Resistor_SMD:R_0603_1608Metric_Pad0.98x0.95mm_HandSolder, F.Cu at (97.5, 162.8)
- added R12: 100k, Resistor_SMD:R_0603_1608Metric_Pad0.98x0.95mm_HandSolder, F.Cu at (97.5, 165.3)
- added R13: 100k, Resistor_SMD:R_0603_1608Metric_Pad0.98x0.95mm_HandSolder, F.Cu at (97.5, 167.8)
- added R14: 100k, Resistor_SMD:R_0603_1608Metric_Pad0.98x0.95mm_HandSolder, F.Cu at (48.9, 117.7)
- added R15: 100k, Resistor_SMD:R_0603_1608Metric_Pad0.98x0.95mm_HandSolder, F.Cu at (48.9, 120.2)
- added R16: 100k, Resistor_SMD:R_0603_1608Metric_Pad0.98x0.95mm_HandSolder, F.Cu at (48.9, 122.7)
- added R17: 100k, Resistor_SMD:R_0603_1608Metric_Pad0.98x0.95mm_HandSolder, F.Cu at (48.9, 125.2)
- added R18: 100k, Resistor_SMD:R_0603_1608Metric_Pad0.98x0.95mm_HandSolder, F.Cu at (48.9, 127.7)
- added R19: 100k, Resistor_SMD:R_0603_1608Metric_Pad0.98x0.95mm_HandSolder, F.Cu at (48.9, 130.2)
- added R2: 100k, Resistor_SMD:R_0603_1608Metric_Pad0.98x0.95mm_HandSolder, F.Cu at (93.2, 162.8)
- added R3: 100k, Resistor_SMD:R_0603_1608Metric_Pad0.98x0.95mm_HandSolder, F.Cu at (93.2, 165.3)
- added R4: 100k, Resistor_SMD:R_0603_1608Metric_Pad0.98x0.95mm_HandSolder, F.Cu at (93.2, 167.8)
- added R5: 100k, Resistor_SMD:R_0603_1608Metric_Pad0.98x0.95mm_HandSolder, B.Cu at (88.0, 124.2)
- added R6: 100k, Resistor_SMD:R_0603_1608Metric_Pad0.98x0.95mm_HandSolder, B.Cu at (104.2, 124.2)
- added R7: 100k, Resistor_SMD:R_0603_1608Metric_Pad0.98x0.95mm_HandSolder, B.Cu at (74.2, 124.6)
- added R8: 100k, Resistor_SMD:R_0603_1608Metric_Pad0.98x0.95mm_HandSolder, F.Cu at (97.5, 155.2)
- added R9: 100k, Resistor_SMD:R_0603_1608Metric_Pad0.98x0.95mm_HandSolder, F.Cu at (97.5, 157.7)
- added RV1: 100kΩ, LCL:TS63X-VISHAY, F.Cu at (98.2, 88.3)
- added S1: PTS526_SK15_SMTR2_LFS, SamacSys_Parts:PTS526SK15SMTR2LFS, F.Cu at (72.5, 86.5)
- added SW1: SW_DIP_x05, Package_DIP:DIP-10_W10.16mm_LongPads, F.Cu at (69.1, 129.8)
- added SW2: SW_DIP_x05, Package_DIP:DIP-10_W10.16mm_LongPads, F.Cu at (85.4, 129.8)
- added SW3: SW_DIP_x05, Package_DIP:DIP-10_W10.16mm_LongPads, F.Cu at (101.7, 129.6)
- added U1: ~, Package_DFN_QFN:QFN-48-1EP_7x7mm_P0.5mm_EP5.15x5.15mm, F.Cu at (103.6, 98.9)
- added U2: ~, Package_TO_SOT_SMD:SOT-23-5_HandSoldering, F.Cu at (97.1, 112.0)

Commit message: Bug correction
Parts:
- removed J14: Conn_Coaxial:60312002114503, Connector_Coaxial:SMA_Wurth_60312002114503_Vertical
- added R20: 1kΩ, Resistor_SMD:R_0603_1608Metric_Pad0.98x0.95mm_HandSolder, B.Cu at (76.0, 92.8)
- added R21: 100kΩ, Resistor_SMD:R_0603_1608Metric_Pad0.98x0.95mm_HandSolder, B.Cu at (76.6, 86.8)
- added R22: 1kΩ, Resistor_SMD:R_0603_1608Metric_Pad0.98x0.95mm_HandSolder, F.Cu at (108.8, 92.0)
- C1, C16, C2, C8, CMR1, COUT1, COUT2, COUT3, R1, R10, R11, R12, R13, R14, R15, R16, R17, R18, R19, R2, R3, R4, R8, R9: moved to B.Cu
- C4: value 100n -> 1µF; moved to B.Cu
- CMaR1: value C -> 10 nF
- LR1: value L -> 21.5 nH
- moved R19 94.2 mm to (123.6, 72.8)
- moved R17 84.1 mm to (114.7, 72.8)
- moved C4 79.8 mm to (76.0, 107.6), turned to -90 degrees
- moved C2 79.2 mm to (76.0, 98.0), turned to -90 degrees
- moved R18 79.2 mm to (105.9, 72.8)
- moved C15 78.2 mm to (109.0, 89.7), turned to 180 degrees
- moved C16 74.4 mm to (108.8, 96.1), turned to -90 degrees
- moved R16 69.4 mm to (97.1, 72.8)
- moved C9 68.0 mm to (115.8, 101.7), turned to -90 degrees
- moved C1 67.5 mm to (98.5, 128.5), turned to 90 degrees
- moved C11 66.4 mm to (111.8, 93.0), turned to 90 degrees
- moved R15 61.4 mm to (87.8, 72.8)
- moved C8 60.2 mm to (76.6, 88.8)
- moved C13 54.4 mm to (108.4, 109.5)
- moved C10 53.5 mm to (101.8, 100.8), turned to 90 degrees
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Connections:
- U1 pad 19: /VS2 -> /VS3
Routing:
- net /VBATT_DVR: track 0.00 -> 38.9 mm
- net /GND: track 0.00 -> 36.7 mm, vias 0 -> 19
- net /VIN2: track 0.00 -> 26.4 mm
- net Net-(S1-NO_1): track 0.00 -> 15.4 mm, vias 0 -> 2
- net /RESET: track 0.00 -> 6.00 mm, vias 0 -> 4
- net /VIN: track 0.00 -> 4.32 mm
- net /DT_D0: track 0.00 -> 3.89 mm
- net /DT_D1: track 0.00 -> 3.82 mm
- net /DT_D4: track 0.00 -> 3.76 mm
- net /DT_D2: track 0.00 -> 3.76 mm
- net /DT_D3: track 0.00 -> 3.75 mm
- added copper zone on B.Cu, net /GND
- added copper zone on In1.Cu, net /GND
- added copper zone on B.Cu, net /RESET
- added copper zone on F.Cu, net /RESET
- added copper zone on B.Cu, net /SW_PULL_UP
- added copper zone on In2.Cu, net /VIN
- added copper zone on In2.Cu, net /VIN2

Commit message: up
Parts:
- C16, CMR1, COUT2: moved to F.Cu
- U1: footprint Package_DFN_QFN:QFN-48-1EP_7x7mm_P0.5mm_EP5.15x5.15mm -> Package_QFP:TQFP-48_7x7mm_P0.5mm
- moved C16 9.69 mm to (109.2, 86.4), turned to 0 degrees
- moved C7 7.04 mm to (106.9, 110.2)
- moved COUT1 4.55 mm to (110.8, 110.0)
- moved LR1 4.50 mm to (112.2, 107.4), turned to 90 degrees
- moved CMaR1 4.47 mm to (115.2, 106.4), turned to -90 degrees
- moved C13 2.79 mm to (107.4, 106.9), turned to -90 degrees
- moved COUT2 2.60 mm to (110.8, 110.0)
- moved CMR1 1.95 mm to (109.6, 107.0), turned to 90 degrees
- moved C6 1.58 mm to (109.2, 92.4)
- moved C11 1.23 mm to (112.1, 91.8)
- moved C15 1.23 mm to (109.3, 88.5)
- moved R22 1.23 mm to (109.2, 90.8)
- moved RV1 0.41 mm to (101.5, 88.6)
Routing:
- net /VDD_IO: track 0.00 -> 79.5 mm, vias 0 -> 6
- net /VBATT: track 0.00 -> 65.3 mm, vias 0 -> 6
- net /DT_D0: track 3.89 -> 67.7 mm, vias 0 -> 1
- net /DT_D1: track 3.82 -> 66.4 mm, vias 0 -> 1
- net /DRIVE_G4: track 0.00 -> 60.7 mm, vias 0 -> 1
- net /DT_D2: track 3.76 -> 64.1 mm, vias 0 -> 1
- net /V1V8O: track 0.00 -> 59.3 mm
- net /SEL_OPEN_LOOP: track 0.00 -> 57.6 mm, vias 0 -> 1
- net /SEL_INT_REF: track 0.00 -> 57.4 mm, vias 0 -> 1
- net /DRIVE_G3: track 0.00 -> 56.9 mm, vias 0 -> 2
- net /DT_D3: track 3.75 -> 59.6 mm, vias 0 -> 1
- net /SEL_CLK: track 0.00 -> 53.7 mm, vias 0 -> 1
- net /ADT_D1: track 0.00 -> 51.9 mm, vias 0 -> 1
- net /ADT_D4: track 0.00 -> 51.4 mm, vias 0 -> 1
- net /EXT_CLK: track 0.00 -> 50.6 mm, vias 0 -> 1
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Other:
- board outline added: 70.5 x 66.6 mm

Commit message: up
Parts:
- moved J1 3.17 mm to (81.8, 72.7)
- moved R15 2.90 mm to (84.9, 72.8)
- moved J2 2.67 mm to (91.6, 72.8)
- moved R16 2.67 mm to (94.4, 72.7)
- moved CLAMP3 2.49 mm to (128.8, 128.2)
- moved COUT3 2.49 mm to (130.6, 125.2)
- moved J9 2.49 mm to (130.8, 118.7)
- moved J4 2.01 mm to (101.0, 72.8)
- moved J12 1.73 mm to (130.8, 109.3)
- moved J3 1.24 mm to (110.5, 72.8)
- moved R17 1.24 mm to (113.4, 72.8)
- moved J13 1.04 mm to (130.8, 100.0)
- moved R19 0.65 mm to (123.0, 72.9)
- moved J5 0.65 mm to (120.1, 72.9)
- moved J8 0.62 mm to (130.7, 90.9)
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Routing:
- net /EXT_CLK: track 50.6 -> 54.4 mm
- net /VG2: track 41.6 -> 43.4 mm
- net /VOUT: track 40.6 -> 42.2 mm
- net /DRIVE_G2: track 41.2 -> 42.3 mm
- net /VG4: track 36.6 -> 37.7 mm
- net /VBATT_PWR: track 49.3 -> 49.9 mm
- net /DRIVE_G3: track 56.9 -> 56.4 mm
- net /SENSE_OSC_CLK: track 35.9 -> 35.8 mm, vias 2 -> 1
Other:
- board size 70.5 x 66.6 mm -> 70.5 x 66.3 mm
