File: MuReSC_BCD_v1/MuReSC_BCD.kicad_sch (KiCad schematic)
At the start: 1 part

Commit message: UP
Parts:
- added C1, C2, C3, C4, C5, C6, C7, CMR (x2), COUT: C, Capacitor_SMD:C_0201_0603Metric_Pad0.64x0.40mm_HandSolder, symbol Device:C
- added CLAMP1, CLAMP2, CLAMP3: 691214110002, SamacSys_Parts:691214110002, symbol SamacSys_Parts:691214110002
- added J1, J10, J11, J12, J14, J2, J3, J4, J5, J6, J7, J8, J9: Conn_Coaxial:60312002114503, Connector_Coaxial:SMA_Wurth_60312002114503_Vertical, symbol Connector:Conn_Coaxial
- added J15: Conn_01x04_Socket, Connector_PinHeader_2.54mm:PinHeader_1x04_P2.54mm_Vertical, symbol Connector:Conn_01x04_Socket
- added JP1, JP2, JP3, JP4, JP5, JP6, JP7: Jumper_3_Open, Connector_PinHeader_2.54mm:PinHeader_1x03_P2.54mm_Vertical, symbol Jumper:Jumper_3_Open
- added LR: L, symbol Device:L
- added R1, R10, R11, R12, R13, R14, R15, R2, R3, R4, R5, R6, R7, R8, R9: 100k, Resistor_SMD:R_0603_1608Metric_Pad0.98x0.95mm_HandSolder, symbol Device:R
- added R16: R_Variable, symbol Device:R_Variable
- added R17: R, symbol Device:R
- added S1: PTS526_SK15_SMTR2_LFS, SamacSys_Parts:PTS526SK15SMTR2LFS, symbol SamacSys_Parts:PTS526_SK15_SMTR2_LFS
- added SW1, SW2, SW3: SW_DIP_x05, Package_DIP:DIP-10_W10.16mm_LongPads, symbol Switch:SW_DIP_x05
- added U2: ~, Package_TO_SOT_SMD:SOT-223, symbol LCL:LD1117AS18TR
Connections:
- net VBATT: now reaches U1.1 (VBATT)
- net VBATT: now also JP3.2 (C), S1.1 (COM_1), S1.2 (COM_2)
- net SEL_DRIVING: now reaches U1.10 (SEL_DRIVING)
- net SEL_DRIVING: now also R11.1, SW3.10
- net VG1: now reaches U1.11 (VG1)
- net VG1: now also J1.1 (In)
- net VG2: now reaches U1.12 (VG2)
- net VG2: now also J2.1 (In)
- net VG3: now reaches U1.13 (VG3)
- net VG3: now also J3.1 (In)
- net VG4: now reaches U1.14 (VG4)
- net VG4: now also J4.1 (In)
- net VBATT_DVR: now reaches U1.15 (VBATT_DRV)
- net VBATT_DVR: now also JP4.2 (C)
- net GND: now reaches U1.16 (GND_IO)
- net GND: now also U1.18 (GND), U1.29 (GND_IO), U1.42 (GND_IO), U1.49 (COOL), U1.6 (GND_IO), C1.2, C2.2, C3.2, C4.2, C5.2, C6.2, C7.2, CLAMP1.2, CLAMP2.2, CLAMP3.2, COUT.2, J1.2 (Ext), J10.2 (Ext), J11.2 (Ext), J12.2 (Ext), J14.2 (Ext), J15.4 (Pin_4), J2.2 (Ext), J3.2 (Ext), J4.2 (Ext), J5.2 (Ext), J6.2 (Ext), J7.2 (Ext), J8.2 (Ext), J9.2 (Ext), R1.2, R10.2, R11.2, R12.2, R13.2, R14.2, R15.2, R16.2, R2.2, R3.2, R4.2, R5.2, R6.2, R7.2, R8.2, R9.2, U2.1 (GND)
- net VDD_IO: now reaches U1.17 (VDD_IO)
- net VDD_IO: now also U1.30 (VDD_IO), U1.43 (VDD_IO), U1.7 (VDD_IO), C3.1, C4.1, C5.1, C6.1, JP2.2 (C)
- net VS2: now reaches U1.19 (VS3)
- net IPTAT_SENSE: now reaches U1.2 (IPTAT_SENSE)
- net IPTAT_SENSE: now also J15.2 (Pin_2)
- net VOUT: now reaches U1.20 (VOUT_SENSE)
- net VOUT: now also U1.21 (VOUT), CLAMP2.1, COUT.1, J10.1 (In), J5.1 (In)
- net VS1: now reaches U1.22 (VS1)
- net VS1: now also CMR.1
- net VBATT_PWR: now reaches U1.23 (VBATT_PWR)
- net VBATT_PWR: now also JP5.2 (C)
- net ADT_D4: now reaches U1.24 (ADT_D4)
- net ADT_D4: now also R10.1, SW2.6
- net ADT_D3: now reaches U1.25 (ADT_D3)
- net ADT_D3: now also R9.1, SW2.7
- net ADT_D2: now reaches U1.26 (ADT_D2)
- net ADT_D2: now also R8.1, SW2.8
- net ADT_D1: now reaches U1.27 (ADT_D1)
- net ADT_D1: now also R7.1, SW2.9
- net ADT_D0: now reaches U1.28 (ADT_D0)
- net ADT_D0: now also R6.1, SW2.10
- net IZTAT_SENSE: now reaches U1.3 (IZTAT_SENSE)
- net IZTAT_SENSE: now also J15.1 (Pin_1)
- net DT_D4: now reaches U1.31 (DT_D4)
- net DT_D4: now also R5.1, SW1.6
- net DT_D3: now reaches U1.32 (DT_D3)
- net DT_D3: now also R4.1, SW1.7
- net DT_D2: now reaches U1.33 (DT_D2)
- net DT_D2: now also R3.1, SW1.8
- net DT_D1: now reaches U1.34 (DT_D1)
- net DT_D1: now also R2.1, SW1.9
- net DT_D0: now reaches U1.35 (DT_D0)
- net DT_D0: now also R1.1, SW1.10
- net EXT_CLK: now reaches U1.36 (EXT_CLK)
- net EXT_CLK: now also J11.1 (In)
- net SEL_CLK: now reaches U1.37 (SEL_CLK)
- net SEL_CLK: now also R12.1, SW3.9
- net SENSE_OSC_CLK: now reaches U1.38 (SENSE_OSC_CLK)
- net SENSE_OSC_CLK: now also J12.1 (In)
- net V1V8: now reaches U1.39 (V1V8)
- net V1V8: now also R17.1, U2.2 (Vout)
- net DRIVE_G1: now reaches U1.4 (DRIVE_G1)
- net DRIVE_G1: now also J6.1 (In)
- net SEL_OPEN_LOOP: now reaches U1.40 (SEL_OPEN_LOOP)
- net SEL_OPEN_LOOP: now also R13.1, SW3.8
- net SENSE_COMP_OUT: now reaches U1.41 (SENSE_CMP_OUT)
- net SENSE_COMP_OUT: now also J14.1 (In)
- net VBATT_COMP: now reaches U1.44 (VBATT_COMP)
- net VBATT_COMP: now also JP6.2 (C)
- net RESET: now reaches U1.45 (RESET)
- net RESET: now also C2.1, R15.1, S1.3 (NO_1), S1.4 (NO_2)
- net SEL_INT_REF: now reaches U1.46 (SEL_INT_REF)
- net SEL_INT_REF: now also R14.1, SW3.7
- net OSC_VCTRL: now reaches U1.47 (OSC_VCTRL)
- net OSC_VCTRL: now also C7.1, R16.1, R17.2
- net EXT_REF_SNS_INT_REF: now reaches U1.48 (EXT_REF_SNS_INT_REF)
- net EXT_REF_SNS_INT_REF: now also J15.3 (Pin_3)
- net DRIVE_G2: now reaches U1.5 (DRIVE_G2)
- net DRIVE_G2: now also J7.1 (In)
- net DRIVE_G3: now reaches U1.8 (DRIVE_G3)
- net DRIVE_G3: now also J8.1 (In)
- net DRIVE_G4: now reaches U1.9 (DRIVE_G4)
- net DRIVE_G4: now also J9.1 (In)
- new net: CMR.1, CMR.2, LR.1
- new net SW_PULL_UP: C1.1, JP1.2 (C), SW1.1, SW1.2, SW1.3, SW1.4, SW1.5, SW2.1, SW2.2, SW2.3, SW2.4, SW2.5, SW3.1, SW3.2, SW3.3, SW3.4, SW3.5
- new net VIN: CLAMP1.1, JP1.1 (A), JP2.1 (A), JP3.1 (A), JP4.1 (A), JP5.1 (A), JP6.1 (A), JP7.1 (A)
- new net VIN2: CLAMP3.1, JP1.3 (B), JP2.3 (B), JP3.3 (B), JP4.3 (B), JP5.3 (B), JP6.3 (B), JP7.3 (B)
- new net VS3: CMR.2, LR.2
- new net V_LDO: JP7.2 (C), U2.3 (VIN)
- no-connect marks 0 -> 8
Other:
- moved on the sheet: U1

Commit message: up
Parts:
- removed R16: R_Variable, symbol Device:R_Variable
- removed U2: ~, Package_TO_SOT_SMD:SOT-223, symbol LCL:LD1117AS18TR
- added C12, C8: 100 nF, Capacitor_SMD:C_0603_1608Metric_Pad1.08x0.95mm_HandSolder, symbol Device:C
- added C14: 10 nF, Capacitor_SMD:C_0603_1608Metric_Pad1.08x0.95mm_HandSolder, symbol Device:C
- added C15: 10 uF, Capacitor_SMD:C_0603_1608Metric_Pad1.08x0.95mm_HandSolder, symbol Device:C
- added C3, C4, C5, C6, C7: 100n, Capacitor_SMD:C_0603_1608Metric_Pad1.08x0.95mm_HandSolder, symbol Device:C
- added COUT2: 1µF, Capacitor_SMD:C_0603_1608Metric_Pad1.08x0.95mm_HandSolder, symbol Device:C
- added COUT3: 10µF, Capacitor_SMD:C_0603_1608Metric_Pad1.08x0.95mm_HandSolder, symbol Device:C
- added JP8: Jumper_3_Open, Connector_PinHeader_2.54mm:PinHeader_1x03_P2.54mm_Vertical, symbol Jumper:Jumper_3_Open
- added R16, R17, R18, R19: 100k, Resistor_SMD:R_0603_1608Metric_Pad0.98x0.95mm_HandSolder, symbol Device:R
- added R20: 1kΩ, symbol Device:R
- added R21: 100kΩ, symbol Device:R
- added RV1: 100kΩ, LCL:TS63X-VISHAY, symbol Device:R_Potentiometer_Trim
- added U2: ~, Package_TO_SOT_SMD:SOT-23-5_HandSoldering, symbol LCL:SPX3819M5-L-1-8-TR
- C1: value C -> 100 nF; footprint Capacitor_SMD:C_0201_0603Metric_Pad0.64x0.40mm_HandSolder -> Capacitor_SMD:C_0603_1608Metric_Pad1.08x0.95mm_HandSolder
- C10: renamed from C4; value C -> 1µF; footprint Capacitor_SMD:C_0201_0603Metric_Pad0.64x0.40mm_HandSolder -> Capacitor_SMD:C_0603_1608Metric_Pad1.08x0.95mm_HandSolder
- C11: renamed from C5; value C -> 1µF; footprint Capacitor_SMD:C_0201_0603Metric_Pad0.64x0.40mm_HandSolder -> Capacitor_SMD:C_0603_1608Metric_Pad1.08x0.95mm_HandSolder
- C13: renamed from C6; value C -> 1µF; footprint Capacitor_SMD:C_0201_0603Metric_Pad0.64x0.40mm_HandSolder -> Capacitor_SMD:C_0603_1608Metric_Pad1.08x0.95mm_HandSolder
- C16: renamed from C7; footprint Capacitor_SMD:C_0201_0603Metric_Pad0.64x0.40mm_HandSolder -> Capacitor_SMD:C_0603_1608Metric_Pad1.08x0.95mm_HandSolder
- C2: value C -> 1µF; footprint Capacitor_SMD:C_0201_0603Metric_Pad0.64x0.40mm_HandSolder -> Capacitor_SMD:C_0603_1608Metric_Pad1.08x0.95mm_HandSolder
- C9: renamed from C3; value C -> 1µF; footprint Capacitor_SMD:C_0201_0603Metric_Pad0.64x0.40mm_HandSolder -> Capacitor_SMD:C_0603_1608Metric_Pad1.08x0.95mm_HandSolder
- CMR1, CMaR1: renamed from CMR; footprint Capacitor_SMD:C_0201_0603Metric_Pad0.64x0.40mm_HandSolder -> Capacitor_SMD:C_0603_1608Metric_Pad1.08x0.95mm_HandSolder
- COUT1: renamed from COUT; value C -> 100nF; footprint Capacitor_SMD:C_0201_0603Metric_Pad0.64x0.40mm_HandSolder -> Capacitor_SMD:C_0603_1608Metric_Pad1.08x0.95mm_HandSolder
- LR1: renamed from LR; footprint (none) -> LCL:Coilcraft-Square-Air-Core-Inductors-all
- R22: renamed from R17; value R -> 1kΩ
- renumbered CLAMP3 to CLAMP2, CLAMP2 to CLAMP3, J11 to J1, J12 to J10, J14 to J11, J4 to J12, J3 to J13, J10 to J14, J6 to J2, J8 to J3, J7 to J4, J9 to J5, J15 to J6, J1 to J7, J2 to J8, J5 to J9, JP3 to JP1, JP7 to JP2, JP4 to JP3, JP1 to JP4, JP2 to JP6, JP6 to JP7, R4 to R10, R9 to R11, R14 to R12, R5 to R13, R10 to R14, R6 to R2, R11 to R3, R2 to R4, R7 to R5, R12 to R6, R3 to R7, R13 to R9
Connections:
- net DRIVE_G1: now also R16.1
- net DRIVE_G2: now also R18.1
- net DRIVE_G3: now also R17.1
- net DRIVE_G4: now also R19.1
- net EXT_CLK: now also R15.1
- net GND: now also C12.2, C14.2, C15.2, C3.2, C4.2, C5.2, C6.2, C7.2, C8.2, COUT2.2, COUT3.2, R16.2, R17.2, R18.2, R19.2, R20.2, RV1.1, U2.2 (GND)
- net OSC_VCTRL: now also RV1.2
- net RESET: now also S1.1 (COM_1), S1.2 (COM_2), C8.1, R21.2; no longer C2.1, R15.1, S1.3 (NO_1), S1.4 (NO_2)
- net V1V8: now also C15.1; no longer U1.39 (V1V8)
- net VBATT: now also C3.1, R21.1; no longer S1.1 (COM_1), S1.2 (COM_2)
- net VBATT_COMP: now also C6.1
- net VBATT_DVR: now also C5.1
- net VBATT_PWR: now also C7.1
- net VIN: now also C2.1
- net VIN2: now also C4.1
- net VOUT: now also COUT2.1, COUT3.1
- net V_LDO: now also C12.1, U2.1 (VIN), U2.3 (EN)
- new net: R20.1, S1.3 (NO_1), S1.4 (NO_2)
- new net: C14.1, U2.4 (BYP)
- new net V1V8I: JP8.3 (B), U2.5 (OUT)
- new net V1V8O: JP8.2 (C), U1.39 (V1V8)
- no-connect marks 8 -> 2
Other:
- moved on the sheet: C10, C11, C13, C16, C9, CLAMP3, COUT1, R22, S1

Commit message: Bug correction
Parts:
- removed J14: Conn_Coaxial:60312002114503, Connector_Coaxial:SMA_Wurth_60312002114503_Vertical, symbol Connector:Conn_Coaxial
- C4: value 100n -> 1µF
- CMaR1: value C -> 10 nF
- LR1: value L -> 21.5 nH
- R20, R21, R22: footprint (none) -> Resistor_SMD:R_0603_1608Metric_Pad0.98x0.95mm_HandSolder
Connections:
- net VS2 is gone; now on net VS3: U1.19 (VS3)
Changed lines of the file:
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@@
   (junction (at 144.78 171.45) (diameter 0) (color 0 0 0 0)
   )
+  (junction (at 162.56 29.21) (diameter 0) (color 0 0 0 0)
+  )
   (junction (at 261.62 30.48) (diameter 0) (color 0 0 0 0)
   )
@@
   (junction (at 182.88 43.18) (diameter 0) (color 0 0 0 0)
   )
-  (junction (at 162.56 29.21) (diameter 0) (color 0 0 0 0)
-  )
   (junction (at 180.34 43.18) (diameter 0) (color 0 0 0 0)
   )
@@
     (stroke (width 0) (type default))
   )
-  (wire (pts (xy 237.49 130.81) (xy 242.57 130.81))
-    (stroke (width 0) (type default))
-  )
   (wire (pts (xy 64.77 21.59) (xy 68.58 21.59))
     (stroke (width 0) (type default))
@@
     (fill (type color) (color 178 178 178 1))
   )
-  (rectangle (start 232.41 124.46) (end 265.43 138.43)
-    (stroke (width -0.0001) (type default))
-    (fill (type color) (color 178 178 178 1))
-  )
   (label "VOUT" (at 251.46 66.04 90) (fields_autoplaced)
     (effects (font (size 1.27 1.27)) (justify left bottom))
@@
     (effects (font (size 1.27 1.27)) (justify left bottom))
   )
-  (label "VOUT" (at 237.49 130.81 0) (fields_autoplaced)
-    (effects (font (size 1.27 1.27)) (justify left bottom))
-  )
   (label "DRIVE_G3" (at 114.3 86.36 0) (fields_autoplaced)
     (effects (font (size 1.27 1.27)) (justify left bottom))
@@
     (effects (font (size 1.27 1.27)) (justify left bottom))
   )
-  (label "VS2" (at 173.99 99.06 0) (fields_autoplaced)
+  (label "VS3" (at 173.99 99.06 0) (fields_autoplaced)
     (effects (font (size 1.27 1.27)) (justify left bottom))
   )
@@
     (effects (font (size 1.27 1.27)) (justify left bottom))
   )
-  (label "GND" (at 247.65 135.89 0) (fields_autoplaced)
-    (effects (font (size 1.27 1.27)) (justify left bottom))
-  )
   (label "GND" (at 152.4 176.53 0) (fields_autoplaced)
     (effects (font (size 1.27 1.27)) (justify left bottom))
@@
     )
   )
-  (symbol (lib_id "Connector:Conn_Coaxial") (at 247.65 130.81 0) (unit 1)
-    (in_bom yes) (on_board yes) (dnp no)
-    (property "Reference" "J14" (at 251.46 129.8332 0)
-      (effects (font (size 1.27 1.27)) (justify left))
-    )
-    (property "Value" "Conn_Coaxial:60312002114503" (at 233.68 127 0)
-      (effects (font (size 1.27 1.27)) (justify left))
-    )
-    (property "Footprint" "Connector_Coaxial:SMA_Wurth_60312002114503_Vertical" (at 247.65 130.81 0)
-      (effects (font (size 1.27 1.27)) hide)
-    )
-    (property "Datasheet" " ~" (at 247.65 130.81 0)
-      (effects (font (size 1.27 1.27)) hide)
-    )
-    (pin "1")
-    (pin "2")
-    (instances
-      (project "MuReSC_BCD"
-        (path "/37ce336a-cad7-4ac4-a72a-85f27d62fb3b"
-          (reference "J14") (unit 1)
-        )
-      )
-    )
-  )
   (symbol (lib_id "Device:R") (at 63.5 187.96 0) (unit 1)
     (in_bom yes) (on_board yes) (dnp no)
@@
     )
   )
-  (symbol (lib_id "Device:R") (at 162.56 25.4 0) (unit 1)
-    (in_bom yes) (on_board yes) (dnp no)
-    (property "Reference" "R21" (at 165.1 24.13 0)
-      (effects (font (size 1.27 1.27)) (justify left))
-    )
-    (property "Value" "100kΩ" (at 165.1 26.67 0)
-      (effects (font (size 1.27 1.27)) (justify left))
-    )
-    (property "Footprint" "" (at 160.782 25.4 90)
-      (effects (font (size 1.27 1.27)) hide)
-    )
-    (property "Datasheet" "~" (at 162.56 25.4 0)
-      (effects (font (size 1.27 1.27)) hide)
-    )
-    (pin "1")
-    (pin "2")
-    (instances
-      (project "MuReSC_BCD"
-        (path "/37ce336a-cad7-4ac4-a72a-85f27d62fb3b"
-          (reference "R21") (unit 1)
-        )
-      )
-    )
-  )
   (symbol (lib_id "Connector:Conn_Coaxial") (at 120.65 184.15 0) (unit 1)
     (in_bom yes) (on_board yes) (dnp no)
@@
       (effects (font (size 1.27 1.27)) (justify left))
     )
-    (property "Value" "C" (at 237.49 69.85 0)
+    (property "Value" "10 nF" (at 237.49 69.85 0)
       (effects (font (size 1.27 1.27)) (justify left))
     )
@@
       (effects (font (size 1.27 1.27)) (justify left))
     )
-    (property "Value" "100n" (at 54.61 35.56 0)
+    (property "Value" "1µF" (at 54.61 35.56 0)
       (effects (font (size 1.27 1.27)) (justify left))
     )
@@
     )
   )
-  (symbol (lib_id "Device:R") (at 269.24 25.4 0) (unit 1)
-    (in_bom yes) (on_board yes) (dnp no)
-    (property "Reference" "R22" (at 271.78 24.13 0)
-      (effects (font (size 1.27 1.27)) (justify left))
-    )
-    (property "Value" "1kΩ" (at 271.78 26.67 0)
-      (effects (font (size 1.27 1.27)) (justify left))
-    )
-    (property "Footprint" "" (at 267.462 25.4 90)
-      (effects (font (size 1.27 1.27)) hide)
-    )
-    (property "Datasheet" "~" (at 269.24 25.4 0)
-      (effects (font (size 1.27 1.27)) hide)
-    )
-    (pin "1")
-    (pin "2")
-    (instances
-      (project "MuReSC_BCD"
-        (path "/37ce336a-cad7-4ac4-a72a-85f27d62fb3b"
-          (reference "R22") (unit 1)
-        )
-      )
-    )
-  )
   (symbol (lib_id "Device:C") (at 223.52 78.74 0) (unit 1)
     (in_bom yes) (on_board yes) (dnp no) (fields_autoplaced)
@@
     )
   )
+  (symbol (lib_id "Device:R") (at 269.24 25.4 0) (unit 1)
+    (in_bom yes) (on_board yes) (dnp no)
+    (property "Reference" "R22" (at 271.78 24.13 0)
+      (effects (font (size 1.27 1.27)) (justify left))
+    )
+    (property "Value" "1kΩ" (at 270.51 26.67 0)
+      (effects (font (size 1.27 1.27)) (justify left))
+    )
+    (property "Footprint" "Resistor_SMD:R_0603_1608Metric_Pad0.98x0.95mm_HandSolder" (at 267.462 25.4 90)
+      (effects (font (size 1.27 1.27)) hide)
+    )
+    (property "Datasheet" "~" (at 269.24 25.4 0)
+      (effects (font (size 1.27 1.27)) hide)
+    )
+    (pin "1")
+    (pin "2")
+    (instances
+      (project "MuReSC_BCD"
+        (path "/37ce336a-cad7-4ac4-a72a-85f27d62fb3b"
+          (reference "R22") (unit 1)
+        )
+      )
+    )
+  )
   (symbol (lib_id "Device:R_Potentiometer_Trim") (at 271.78 36.83 180) (unit 1)
     (in_bom yes) (on_board yes) (dnp no) (fields_autoplaced)
@@
       (effects (font (size 1.27 1.27)) (justify left))
     )
-    (property "Value" "L" (at 234.95 80.01 0)
+    (property "Value" "21.5 nH" (at 234.95 80.01 0)
       (effects (font (size 1.27 1.27)) (justify left))
     )
@@
     )
   )
-  (symbol (lib_id "Device:R") (at 147.32 48.26 90) (unit 1)
-    (in_bom yes) (on_board yes) (dnp no)
-    (property "Reference" "R20" (at 146.05 45.72 0)
-      (effects (font (size 1.27 1.27)) (justify left))
-    )
-    (property "Value" "1kΩ" (at 148.59 45.72 0)
-      (effects (font (size 1.27 1.27)) (justify left))
-    )
-    (property "Footprint" "" (at 147.32 50.038 90)
-      (effects (font (size 1.27 1.27)) hide)
-    )
-    (property "Datasheet" "~" (at 147.32 48.26 0)
-      (effects (font (size 1.27 1.27)) hide)
-    )
-    (pin "1")
-    (pin "2")
-    (instances
-      (project "MuReSC_BCD"
-        (path "/37ce336a-cad7-4ac4-a72a-85f27d62fb3b"
-          (reference "R20") (unit 1)
-        )
-      )
-    )
-  )
   (symbol (lib_id "Jumper:Jumper_3_Open") (at 74.93 21.59 0) (unit 1)
     (in_bom yes) (on_board yes) (dnp no) (fields_autoplaced)
@@
     )
   )
+  (symbol (lib_id "Device:R") (at 162.56 25.4 0) (unit 1)
+    (in_bom yes) (on_board yes) (dnp no)
+    (property "Reference" "R21" (at 165.1 24.13 0)
+      (effects (font (size 1.27 1.27)) (justify left))
+    )
+    (property "Value" "100kΩ" (at 163.83 26.67 0)
+      (effects (font (size 1.27 1.27)) (justify left))
+    )
+    (property "Footprint" "Resistor_SMD:R_0603_1608Metric_Pad0.98x0.95mm_HandSolder" (at 160.782 25.4 90)
+      (effects (font (size 1.27 1.27)) hide)
+    )
+    (property "Datasheet" "~" (at 162.56 25.4 0)
+      (effects (font (size 1.27 1.27)) hide)
+    )
+    (pin "1")
+    (pin "2")
+    (instances
+      (project "MuReSC_BCD"
+        (path "/37ce336a-cad7-4ac4-a72a-85f27d62fb3b"
+          (reference "R21") (unit 1)
+        )
+      )
+    )
+  )
   (symbol (lib_id "Device:C") (at 21.59 118.11 0) (unit 1)
     (in_bom yes) (on_board yes) (dnp no) (fields_autoplaced)
@@
         )
       )
+    )
+  )
+  (symbol (lib_id "Device:R") (at 147.32 48.26 90) (unit 1)
+    (in_bom yes) (on_board yes) (dnp no)
+    (property "Reference" "R20" (at 146.05 45.72 0)
+      (effects (font (size 1.27 1.27)) (justify left))
+    )
+    (property "Value" "1kΩ" (at 148.59 46.99 0)
+      (effects (font (size 1.27 1.27)) (justify left))
+    )
+    (property "Footprint" "Resistor_SMD:R_0603_1608Metric_Pad0.98x0.95mm_HandSolder" (at 147.32 50.038 90)
+      (effects (font (size 1.27 1.27)) hide)
+    )
+    (property "Datasheet" "~" (at 147.32 48.26 0)
+      (effects (font (size 1.27 1.27)) hide)
+    )
+    (pin "1")
+    (pin "2")
+    (instances
+      (project "MuReSC_BCD"
+        (path "/37ce336a-cad7-4ac4-a72a-85f27d62fb3b"
+          (reference "R20") (unit 1)
+        )
+      )

Commit message: up
Parts:
- U1: footprint Package_DFN_QFN:QFN-48-1EP_7x7mm_P0.5mm_EP5.15x5.15mm -> Package_QFP:TQFP-48_7x7mm_P0.5mm
Connections:
- net GND: no longer U1.49 (COOL)
Changed lines of the file:
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@@
   (junction (at 86.36 105.41) (diameter 0) (color 0 0 0 0)
-  )
-  (junction (at 160.02 142.24) (diameter 0) (color 0 0 0 0)
   )
   (junction (at 63.5 132.08) (diameter 0) (color 0 0 0 0)
@@
   )
   (wire (pts (xy 34.29 102.87) (xy 39.37 102.87))
-    (stroke (width 0) (type default))
-  )
-  (wire (pts (xy 160.02 135.89) (xy 160.02 142.24))
     (stroke (width 0) (type default))
   )
@@
       (effects (font (size 1.27 1.27)))
     )
-    (property "Footprint" "Package_DFN_QFN:QFN-48-1EP_7x7mm_P0.5mm_EP5.15x5.15mm" (at 153.67 101.6 0)
+    (property "Footprint" "Package_QFP:TQFP-48_7x7mm_P0.5mm" (at 153.67 101.6 0)
       (effects (font (size 1.27 1.27)) hide)
     )
@@
     (pin "47")
     (pin "48")
-    (pin "49")
     (pin "5")
     (pin "6")

Commit message: up
Parts:
- C16: value C -> 1u
Changed lines of the file:
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@@
       (effects (font (size 1.27 1.27)) (justify left))
     )
-    (property "Value" "C" (at 265.43 36.83 0)
+    (property "Value" "1u" (at 265.43 36.83 0)
       (effects (font (size 1.27 1.27)) (justify left))
     )
